File: Open2327RomAdapter.kicad_pcb (KiCad board)
At the start: 2 copper layers, 19.6 x 41.5 mm, 10 parts, among them J1 CONN_A12, P1 Conn_01x04, P99 OSHW_LOGO, U1 2364_SOCKET, U2 27128

Commit message: Version 3.1
Parts:
- removed P1: Conn_01x04, Open2327RomAdapter:Solderable_PinHeader_1x04
- added JP2: J_A14, TestPoint:TestPoint_2Pads_Pitch2.54mm_Drill0.8mm, F.Cu at (156.0, 97.5)
- added JP3: J_A15, TestPoint:TestPoint_2Pads_Pitch2.54mm_Drill0.8mm, F.Cu at (161.0, 97.5)
- added JP4: J_A12, TestPoint:TestPoint_2Pads_Pitch2.54mm_Drill0.8mm, F.Cu at (146.3, 100.1)
- added JP5: JUMPER_4K_SW, Jumper:SolderJumper-2_P1.3mm_Bridged_RoundedPad1.0x1.5mm, B.Cu at (155.7, 121.2)
- JP1: value JUMPER_4K_SW -> J_A13; footprint Jumper:SolderJumper-2_P1.3mm_Bridged_RoundedPad1.0x1.5mm -> TestPoint:TestPoint_2Pads_Pitch2.54mm_Drill0.8mm; moved to F.Cu
- P99: moved to F.Cu
- R1, R2, R3, R4: footprint Resistor_SMD:R_0805_2012Metric_Pad1.15x1.40mm_HandSolder -> Resistor_THT:R_Axial_DIN0207_L6.3mm_D2.5mm_P10.16mm_Horizontal
- moved JP1 18.4 mm to (150.9, 97.5)
- moved P99 0.13 mm to (154.7, 132.1), turned to 90 degrees
Connections:
- JP1 pad 1: Net-(J1-Pad1) -> Net-(JP1-Pad1)
- JP1 pad 2: Net-(JP1-Pad2) -> GND
- R1 pad 1: Net-(P1-Pad4) -> Net-(JP1-Pad1)
- U1 pad 21: Net-(JP1-Pad2) -> Net-(JP5-Pad2)
- U2 pad 26: Net-(P1-Pad4) -> Net-(JP1-Pad1)
Routing:
- net Net-(JP1-Pad1): track 0.00 -> 22.3 mm
- net Net-(P1-Pad4): track 17.1 -> 0.00 mm, vias 1 -> 0
- net Net-(JP5-Pad2): track 0.00 -> 13.1 mm
- net VCC: track 16.5 -> 24.4 mm
- net Net-(J1-Pad1): track 24.1 -> 27.7 mm, vias 1 -> 0
- net Net-(JP3-Pad1): track 23.9 -> 20.8 mm, vias 0 -> 1
- net Net-(JP1-Pad2): track 2.40 -> 0.00 mm
- net Net-(JP2-Pad1): track 18.2 -> 17.1 mm, vias 0 -> 1
- net Net-(U1-Pad18): track 11.4 -> 10.6 mm
Other:
- board text added: "A13"
- board text added: "A14"
- board text added: "A15"
- board text added: "V3.1"
- board text added: "https://github.com/nharrer/ Open2327RomAdapter"
- board text removed: "GND A15 A14 A13"
- board text removed: "V3"
- board text removed: "github.com/SukkoPera/Open2327RomAdapter"
